Commit message: in between

File: workspace/puma560_ros2_moveit/src/puma560_description/urdf/puma560_robot.urdf (robot description, URDF)
Before this commit: robot puma560, 8 links, 7 joints
Links:
- added link lift_column_link; visual box size=0.08 0.08 1.2; visual box size=0.4 0.4 0.02
- added link lift_link; collision box size=0.25 0.25 0.05; visual box size=0.12 0.1 0.15
Joints:
- removed joint virtual_joint
- added joint arm_base_joint: type fixed, parent lift_link, child link1, origin xyz=0 0 0 rpy=0 0 0
- added joint lift_column_joint: type fixed, parent world, child lift_column_link, origin xyz=0 0 0 rpy=0 0 0
- added joint lift_joint: type prismatic, parent world, child lift_link, origin xyz=0 0 0 rpy=0 0 0, axis 0 0 1, limit lower=0.0 upper=1.0 effort=5000.0 velocity=1.0
- joint j1: limit lower=-3.14159265 upper=3.14159265 effort=1000.0 velocity=0 -> lower=-3.14159265 upper=3.14159265 effort=1000.0 velocity=2.0
- joint j2: limit lower=-1.570796325 upper=1.570796325 effort=1000.0 velocity=0 -> lower=-1.570796325 upper=1.570796325 effort=1000.0 velocity=2.0
- joint j3: limit lower=-1.570796325 upper=1.570796325 effort=1000.0 velocity=0 -> lower=-1.570796325 upper=1.570796325 effort=1000.0 velocity=2.0
- joint j4: limit lower=-1.570796325 upper=1.570796325 effort=1000.0 velocity=0 -> lower=-1.570796325 upper=1.570796325 effort=1000.0 velocity=2.0
- joint j5: limit lower=-1.570796325 upper=1.570796325 effort=1000.0 velocity=0 -> lower=-1.570796325 upper=1.570796325 effort=1000.0 velocity=2.0
- joint j6: limit lower=-1.570796325 upper=1.570796325 effort=1000.0 velocity=0 -> lower=-1.570796325 upper=1.570796325 effort=1000.0 velocity=2.0

File: workspace/puma560_ros2_moveit/src/puma560_description/urdf/puma560_robot_gazebo.xacro (robot description, xacro)
@@ -16,3 +16,42 @@
     </xacro:unless>
   </gazebo>
+  <!-- Gazebo joint physics settings for lift_joint -->
+  <gazebo reference="lift_joint">
+    <provideFeedback>true</provideFeedback>
+    <implicitSpringDamper>true</implicitSpringDamper>
+  </gazebo>
+  <!-- ========== LIFT MECHANISM COLLISION SETTINGS ========== -->
+  <!-- Lift column (fixed structure) - no collision to allow lift movement -->
+  <gazebo reference="lift_column_link">
+    <selfCollide>false</selfCollide>
+  </gazebo>
+  <!-- Lift platform (moving carriage) -->
+  <gazebo reference="lift_link">
+    <mu1>0.2</mu1>
+    <mu2>0.2</mu2>
+    <selfCollide>false</selfCollide>
+  </gazebo>
+  <!-- ========== ARM LINKS COLLISION SETTINGS ========== -->
+  <!-- Disable self-collision for all arm links to prevent internal collisions -->
+  <gazebo reference="link1">
+    <selfCollide>false</selfCollide>
+  </gazebo>
+  <gazebo reference="link2">
+    <selfCollide>false</selfCollide>
+  </gazebo>
+  <gazebo reference="link3">
+    <selfCollide>false</selfCollide>
+  </gazebo>
+  <gazebo reference="link4">
+    <selfCollide>false</selfCollide>
+  </gazebo>
+  <gazebo reference="link5">
+    <selfCollide>false</selfCollide>
+  </gazebo>
+  <gazebo reference="link6">
+    <selfCollide>false</selfCollide>
+  </gazebo>
+  <gazebo reference="link7">
+    <selfCollide>false</selfCollide>
+  </gazebo>
 </robot>

File: workspace/puma560_ros2_moveit/src/puma560_description/urdf/puma560_robot_ros2_control.xacro (robot description, xacro)
@@ -16,4 +16,13 @@
             </hardware>
         </xacro:unless>
+        <!-- Lift Joint (Prismatic - Z axis, 0 to 1 meter) -->
+        <joint name="lift_joint">
+            <command_interface name="position">
+                <param name="min">0.0</param>
+                <param name="max">1.0</param>
+            </command_interface>
+            <state_interface name="position"/>
+            <state_interface name="velocity"/>
+        </joint>
         <joint name="j1">
             <command_interface name="position">
